File: hardware/Penguino-STM32WL-LoRa-E5/Penguino-STM32WL-LoRa-E5.sch (KiCad schematic (older format))
At the start: 56 parts, among them J1 JST_PH, J2 USB_C_Receptacle_USB2.0, J3 Conn_ARM_JTAG_SWD_10, J4 U.FL/iPEX, J5 SMA-Edge-Mount, Q1 NCE3407A, SW1 RESET, SW2 USR_BTN, U1 MCP73831, U2 RT9078-33GJ5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

Commit message: fix: NRST and USB Footprint
Parts:
- J2: footprint Connector_USB:USB_C_Receptacle_Palconn_UTC16-G -> Connector_USB:USB_C_Receptacle_HRO_TYPE-C-31-M-12
Connections:
- net NRST is gone; now on net RST: J3.10 (~RESET~)
Changed lines of the file:
@@
 Title "Penguino STM32WL LoRa-E5"
 Date "2020-11-24"
-Rev "0.1"
+Rev "0.2"
 Comp "Makertronika Labs"
 Comment1 "https://makertronika.com/"
@@
 F 0 "J2" H 625 2975 50  0000 C CNN
 F 1 "USB_C_Receptacle_USB2.0" H 1182 3826 50  0000 C CNN
-F 2 "Connector_USB:USB_C_Receptacle_Palconn_UTC16-G" H 1225 3050 50  0001 C CNN
+F 2 "Connector_USB:USB_C_Receptacle_HRO_TYPE-C-31-M-12" H 1225 3050 50  0001 C CNN
 F 3 "https://www.usb.org/sites/default/files/documents/usb_type-c.zip" H 1225 3050 50  0001 C CNN
 F 4 "TYPE-C-31-M-12" H 1075 3050 50  0001 C CNN "MPN"
@@
 Wire Notes Line
 	6550 6475 8750 6475
-Text GLabel 3150 5175 2    50   Input ~ 0
-NRST
 Text GLabel 6025 3775 2    50   Input ~ 0
 RST
@@
 Wire Wire Line
 	7850 5025 7900 5025
+Text GLabel 3150 5175 2    50   Input ~ 0
+RST
 $EndSCHEMATC
